Commit message: new: working control simulation

File: src/roboarm_description/urdf/roboarm.urdf.xacro (robot description, xacro)
@@ -1,3 +1,7 @@
 <robot name="roboarm" xmlns:xacro="http://www.ros.org/wiki/xacro">
+    <!-- Include Gazebo Parameters -->
+    <xacro:include filename="$(find roboarm_description)/urdf/roboarm_gazebo.xacro" />
+    <!-- Include ros2_control Plugins -->
+    <xacro:include filename="$(find roboarm_description)/urdf/roboarm_ros2_control.xacro" />
     <!-- Xacro properties -->
     <xacro:property name="base_length" value="0.5" />
@@ -84,5 +88,6 @@
     </material>
     <!-- Links -->
-    <link name="base_dummy_link" />
+    <!-- <link name="base_dummy_link" /> -->
+    <link name="world"/>
     <!-- Making base_link -->
     <xacro:box_link name="base" x="${base_length}" y="${base_length}" z="${base_height}" ox="0" oy="0" oz="${base_height  / 2}" mass="10" material="black" />
@@ -110,6 +115,6 @@
     <xacro:box_link name="right_finger" x="${arm_width * 0.5}" y="${arm_width * 0.5}" z="${arm_width * 4}" ox="0" oy="0" oz="${arm_width * 4 / 2}" mass="0.02" material="orange" />
     <!-- Joints -->
-    <joint name="dummy_base_joint" type="fixed">
-        <parent link="base_dummy_link" />
+    <joint name="world_base_joint" type="fixed">
+        <parent link="world" />
         <child link="base_link" />
         <origin xyz="0 0 0" rpy="0 0 0" />
@@ -120,5 +125,5 @@
         <origin xyz="0 0 ${base_height}" rpy="0 0 0" />
         <axis xyz="0 0 1" />
-        <limit lower="${-pi}" upper="${pi}" velocity="100" effort="100"/>
+        <limit lower="${-pi}" upper="${pi}" velocity="2.0" effort="100"/>
     </joint>
     <joint name="body_root1_joint" type="revolute">
@@ -127,5 +132,5 @@
         <origin xyz="0 ${body_radius} ${body_length - root_radius}" rpy="0 0 0" />
         <axis xyz="0 1 0" />
-        <limit lower="${-pi}" upper="${pi}" velocity="100" effort="100"/>
+        <limit lower="${-pi}" upper="${pi}" velocity="2.0" effort="100"/>
     </joint>
     <joint name="root1_shoulder_joint" type="fixed">
@@ -139,5 +144,5 @@
         <origin xyz="0 0 ${arm_length - (2 * root_radius)}" rpy="0 0 0" />
         <axis xyz="0 1 0" />
-        <limit lower="${-pi}" upper="${pi}" velocity="100" effort="100"/>
+        <limit lower="${-pi}" upper="${pi}" velocity="2.0" effort="100"/>
     </joint>
     <joint name="root2_forearm_joint" type="fixed">
@@ -151,5 +156,5 @@
         <origin xyz="0 0 ${arm_length - (2 * root_radius)}" rpy="0 0 0" />
         <axis xyz="0 1 0" />
-        <limit lower="${-pi}" upper="${pi}" velocity="100" effort="100"/>
+        <limit lower="${-pi}" upper="${pi}" velocity="2.0" effort="100"/>
     </joint>
     <joint name="root3_wrist_joint" type="fixed">
@@ -163,5 +168,5 @@
         <origin xyz="0 ${arm_width / 2} ${(arm_length * 0.5) - root_radius}" rpy="0 0 0" />
         <axis xyz="0 0 1" />
-        <limit lower="${-pi}" upper="${pi}" velocity="100" effort="100"/>
+        <limit lower="${-pi}" upper="${pi}" velocity="2.0" effort="100"/>
     </joint>
     <joint name="root4_palm_joint" type="fixed">
@@ -175,5 +180,5 @@
         <origin xyz="${(-arm_width * 3 / 2) + (arm_width * 0.5 / 2)} 0 ${arm_width}" rpy="0 0 0" />
         <axis xyz="1 0 0" />
-        <limit lower="0" upper="${(arm_width * 3 / 2) - (arm_width * 0.5)}" velocity="100" effort="100"/>
+        <limit lower="0" upper="${(arm_width * 3 / 2) - (arm_width * 0.5)}" velocity="2.0" effort="100"/>
     </joint>
     <joint name="palm_right_finger_joint" type="prismatic">
@@ -182,5 +187,6 @@
         <origin xyz="${(arm_width * 3 / 2) - (arm_width * 0.5 / 2)} 0 ${arm_width}" rpy="0 0 0" />
         <axis xyz="1 0 0" />
-        <limit lower="${-(arm_width * 3 / 2) + (arm_width * 0.5)}" upper="0" velocity="100" effort="100"/>
+        <limit lower="${-(arm_width * 3 / 2) + (arm_width * 0.5)}" upper="0" velocity="2.0" effort="100"/>
+        <mimic joint="palm_left_finger_joint" multiplier="-1" />
     </joint>
 </robot>

Commit message: fix: experiments

File: src/roboarm_description/urdf/roboarm.urdf.xacro (robot description, xacro)
@@ -11,6 +11,10 @@
     <xacro:property name="root_radius" value="0.05" />
     <xacro:property name="root_length" value="0.05" />
+    <xacro:property name="root_mass" value="0.001" />
     <xacro:property name="arm_width" value="0.05" />
     <xacro:property name="arm_length" value="0.5" />
+    <xacro:property name="arm_mass" value="0.01" />
+    <xacro:property name="damping" value="0.0" />
+    <xacro:property name="friction" value="0.0" />
     <!-- Xacro macros -->
     <xacro:macro name="cylinder_link" params="name r l ox oy oz oroll opitch oyaw mass material">
@@ -68,4 +72,22 @@
         </inertial>
     </xacro:macro>
+    <!-- <xacro:macro name="box_inertia" params="m x y z o_xyz o_rpy">
+        <inertial>
+        <mass value="${m}" />
+        <origin xyz="0 0 0" rpy="0 0 0" />
+        <inertia ixx="1.0" ixy="0" ixz="0"
+                 iyy="1.0" iyz="0"
+                 izz="1.0" />
+        </inertial>
+    </xacro:macro>
+    <xacro:macro name="cylinder_inertia" params="m r l o_xyz o_rpy">
+        <inertial>
+            <mass value="${m}" />
+            <origin xyz="0 0 0" rpy="0 0 0" />
+            <inertia ixx="1.0" ixy="0" ixz="0"
+                     iyy="1.0" iyz="0"
+                     izz="1.0" />
+        </inertial>
+    </xacro:macro>
     <xacro:macro name="sphere_inertia" params="m r o_xyz o_rpy">
         <inertial>
@@ -76,5 +98,5 @@
                      izz="${(2/5) * m * r * r}" />
         </inertial>
-    </xacro:macro>
+    </xacro:macro> -->
     <!-- Materials -->
     <material name="black">
@@ -95,23 +117,23 @@
     <xacro:cylinder_link name="body" r="${body_radius}" l="${body_length}" ox="0" oy="0" oz="${body_length / 2}" oroll="0" opitch="0" oyaw="0" mass="5.0" material="orange" />
     <!-- Making root1_link -->
-    <xacro:cylinder_link name="root1" r="${root_radius}" l="${root_length}" ox="0" oy="${root_length / 2}" oz="0" oroll="${pi / 2}" opitch="0" oyaw="0" mass="0.1" material="gray" />
+    <xacro:cylinder_link name="root1" r="${root_radius}" l="${root_length}" ox="0" oy="${root_length / 2}" oz="0" oroll="${pi / 2}" opitch="0" oyaw="0" mass="${root_mass}" material="gray" />
     <!-- Making shoulder link -->
-    <xacro:box_link name="shoulder" x="${arm_width}" y="${arm_width}" z="${arm_length}" ox="0" oy="${arm_width / 2}" oz="${(arm_length / 2) - root_radius}" mass="0.2" material="orange" />
+    <xacro:box_link name="shoulder" x="${arm_width}" y="${arm_width}" z="${arm_length}" ox="0" oy="${arm_width / 2}" oz="${(arm_length / 2) - root_radius}" mass="${arm_mass}" material="orange" />
     <!-- Making root2_link -->
-    <xacro:cylinder_link name="root2" r="${root_radius}" l="${root_length}" ox="0" oy="${-root_length / 2}" oz="0" oroll="${pi / 2}" opitch="0" oyaw="0" mass="0.1" material="gray" />
+    <xacro:cylinder_link name="root2" r="${root_radius}" l="${root_length}" ox="0" oy="${-root_length / 2}" oz="0" oroll="${pi / 2}" opitch="0" oyaw="0" mass="${root_mass}" material="gray" />
     <!-- Making forearm_link -->
-    <xacro:box_link name="forearm" x="${arm_width}" y="${arm_width}" z="${arm_length}" ox="0" oy="${-arm_width / 2}" oz="${(arm_length / 2) - root_radius}" mass="0.2" material="orange" />
+    <xacro:box_link name="forearm" x="${arm_width}" y="${arm_width}" z="${arm_length}" ox="0" oy="${-arm_width / 2}" oz="${(arm_length / 2) - root_radius}" mass="${arm_mass}" material="orange" />
     <!-- Making root3_link -->
-    <xacro:cylinder_link name="root3" r="${root_radius}" l="${root_length}" ox="0" oy="${root_length / 2}" oz="0" oroll="${pi / 2}" opitch="0" oyaw="0" mass="0.1" material="gray" />
+    <xacro:cylinder_link name="root3" r="${root_radius}" l="${root_length}" ox="0" oy="${root_length / 2}" oz="0" oroll="${pi / 2}" opitch="0" oyaw="0" mass="${root_mass}" material="gray" />
     <!-- Making wrist_link -->
-    <xacro:box_link name="wrist" x="${arm_width}" y="${arm_width}" z="${arm_length / 2}" ox="0" oy="${arm_width / 2}" oz="${(arm_length / 4) - root_radius}" mass="0.1" material="orange" />
+    <xacro:box_link name="wrist" x="${arm_width}" y="${arm_width}" z="${arm_length / 2}" ox="0" oy="${arm_width / 2}" oz="${(arm_length / 4) - root_radius}" mass="${arm_mass}" material="orange" />
     <!-- Making root4_link -->
-    <xacro:cylinder_link name="root4" r="${root_radius}" l="${root_length}" ox="0" oy="0" oz="${root_length / 2}" oroll="0" opitch="0" oyaw="0" mass="0.1" material="gray" />
+    <xacro:cylinder_link name="root4" r="${root_radius}" l="${root_length}" ox="0" oy="0" oz="${root_length / 2}" oroll="0" opitch="0" oyaw="0" mass="${root_mass}" material="gray" />
     <!-- Making palm link -->
-    <xacro:box_link name="palm" x="${arm_width * 3}" y="${arm_width}" z="${arm_width}" ox="0" oy="0" oz="${arm_width / 2}" mass="0.05" material="orange" />
+    <xacro:box_link name="palm" x="${arm_width * 3}" y="${arm_width}" z="${arm_width}" ox="0" oy="0" oz="${arm_width / 2}" mass="${arm_mass}" material="orange" />
     <!-- Making left_finger_link -->
-    <xacro:box_link name="left_finger" x="${arm_width * 0.5}" y="${arm_width * 0.5}" z="${arm_width * 4}" ox="0" oy="0" oz="${arm_width * 4 / 2}" mass="0.02" material="orange" />
+    <xacro:box_link name="left_finger" x="${arm_width * 0.5}" y="${arm_width * 0.5}" z="${arm_width * 4}" ox="0" oy="0" oz="${arm_width * 4 / 2}" mass="0.001" material="orange" />
     <!-- Making right_finger_link -->
-    <xacro:box_link name="right_finger" x="${arm_width * 0.5}" y="${arm_width * 0.5}" z="${arm_width * 4}" ox="0" oy="0" oz="${arm_width * 4 / 2}" mass="0.02" material="orange" />
+    <xacro:box_link name="right_finger" x="${arm_width * 0.5}" y="${arm_width * 0.5}" z="${arm_width * 4}" ox="0" oy="0" oz="${arm_width * 4 / 2}" mass="0.001" material="orange" />
     <!-- Joints -->
     <joint name="world_base_joint" type="fixed">
@@ -125,6 +147,24 @@
         <origin xyz="0 0 ${base_height}" rpy="0 0 0" />
         <axis xyz="0 0 1" />
-        <limit lower="${-pi}" upper="${pi}" velocity="2.0" effort="100"/>
-    </joint>
+        <dynamics damping="${damping}" friction="${friction}"/>
+        <limit lower="${-pi / 2}" upper="${pi / 2}" velocity="2.0" effort="100"/>
+    </joint>
+    <transmission name="base_body_joint_trans">
+        <type>transmission_interface/SimpleTransmission</type>
+        <joint name="base_body_joint">
+          <hardwareInterface>hardware_interface/EffortJointInterface</hardwareInterface>
+        </joint>
+        <actuator name="base_body_joint_motor">
+          <hardwareInterface>hardware_interface/EffortJointInterface</hardwareInterface>
+          <mechanicalReduction>1</mechanicalReduction>
+        </actuator>
+    </transmission>
+    <!-- <transmission name="base_body_joint_trans">
+        <plugin>transmission_interface/SimpleTransmission</plugin>
+        <actuator name="motor_base_body_joint" role="actuator1" />
+        <joint name="base_body_joint" role="joint1">
+            <mechanical_reduction>1.0</mechanical_reduction>
+        </joint>
+    </transmission> -->
     <joint name="body_root1_joint" type="revolute">
         <parent link="body_link" />
@@ -132,6 +172,24 @@
         <origin xyz="0 ${body_radius} ${body_length - root_radius}" rpy="0 0 0" />
         <axis xyz="0 1 0" />
-        <limit lower="${-pi}" upper="${pi}" velocity="2.0" effort="100"/>
-    </joint>
+        <limit lower="${-pi / 4}" upper="${pi / 4}" velocity="2.0" effort="100"/>
+        <dynamics damping="${damping}" friction="${friction}"/>
+    </joint>
+    <transmission name="body_root1_joint_trans">
+        <type>transmission_interface/SimpleTransmission</type>
+        <joint name="body_root1_joint">
+          <hardwareInterface>hardware_interface/EffortJointInterface</hardwareInterface>
+        </joint>
+        <actuator name="body_root1_joint_motor">
+          <hardwareInterface>hardware_interface/EffortJointInterface</hardwareInterface>
+          <mechanicalReduction>1</mechanicalReduction>
+        </actuator>
+    </transmission>
+    <!-- <transmission name="body_root1_joint_trans">
+        <plugin>transmission_interface/SimpleTransmission</plugin>
+        <actuator name="motor_body_root1_joint" role="actuator1" />
+        <joint name="body_root1_joint" role="joint1">
+            <mechanical_reduction>1.0</mechanical_reduction>
+        </joint>
+    </transmission> -->
     <joint name="root1_shoulder_joint" type="fixed">
         <parent link="root1_link" />
@@ -144,6 +202,24 @@
         <origin xyz="0 0 ${arm_length - (2 * root_radius)}" rpy="0 0 0" />
         <axis xyz="0 1 0" />
-        <limit lower="${-pi}" upper="${pi}" velocity="2.0" effort="100"/>
-    </joint>
+        <limit lower="${-pi / 4}" upper="${pi / 4}" velocity="2.0" effort="100"/>
+        <dynamics damping="${damping}" friction="${friction}"/>
+    </joint>
+    <transmission name="shoulder_root2_joint_trans">
+        <type>transmission_interface/SimpleTransmission</type>
+        <joint name="shoulder_root2_joint">
+          <hardwareInterface>hardware_interface/EffortJointInterface</hardwareInterface>
+        </joint>
+        <actuator name="shoulder_root2_joint_motor">
+          <hardwareInterface>hardware_interface/EffortJointInterface</hardwareInterface>
+          <mechanicalReduction>1</mechanicalReduction>
+        </actuator>
+    </transmission>
+    <!-- <transmission name="shoulder_root2_joint_trans">
+        <plugin>transmission_interface/SimpleTransmission</plugin>
+        <actuator name="motor_shoulder_root2_joint" role="actuator1" />
+        <joint name="shoulder_root2_joint" role="joint1">
+            <mechanical_reduction>1.0</mechanical_reduction>
+        </joint>
+    </transmission> -->
     <joint name="root2_forearm_joint" type="fixed">
         <parent link="root2_link" />
@@ -156,6 +232,24 @@
         <origin xyz="0 0 ${arm_length - (2 * root_radius)}" rpy="0 0 0" />
         <axis xyz="0 1 0" />
-        <limit lower="${-pi}" upper="${pi}" velocity="2.0" effort="100"/>
-    </joint>
+        <limit lower="${-pi / 4}" upper="${pi / 4}" velocity="2.0" effort="100"/>
+        <dynamics damping="${damping}" friction="${friction}"/>
+    </joint>
+    <transmission name="forearm_root3_joint_trans">
+        <type>transmission_interface/SimpleTransmission</type>
+        <joint name="forearm_root3_joint">
+          <hardwareInterface>hardware_interface/EffortJointInterface</hardwareInterface>
+        </joint>
+        <actuator name="forearm_root3_joint_motor">
+          <hardwareInterface>hardware_interface/EffortJointInterface</hardwareInterface>
+          <mechanicalReduction>1</mechanicalReduction>
+        </actuator>
+    </transmission>
+    <!-- <transmission name="forearm_root3_joint_trans">
+        <plugin>transmission_interface/SimpleTransmission</plugin>
+        <actuator name="forearm_root3_joint_joint" role="actuator1" />
+        <joint name="forearm_root3_joint" role="joint1">
+            <mechanical_reduction>1.0</mechanical_reduction>
+        </joint>
+    </transmission> -->
     <joint name="root3_wrist_joint" type="fixed">
         <parent link="root3_link" />
@@ -168,6 +262,24 @@
         <origin xyz="0 ${arm_width / 2} ${(arm_length * 0.5) - root_radius}" rpy="0 0 0" />
         <axis xyz="0 0 1" />
-        <limit lower="${-pi}" upper="${pi}" velocity="2.0" effort="100"/>
-    </joint>
+        <limit lower="${-pi / 2}" upper="${pi / 2}" velocity="2.0" effort="100"/>
+        <dynamics damping="${damping}" friction="${friction}"/>
+    </joint>
+    <transmission name="wrist_root4_joint_trans">
+        <type>transmission_interface/SimpleTransmission</type>
+        <joint name="wrist_root4_joint">
+          <hardwareInterface>hardware_interface/EffortJointInterface</hardwareInterface>
+        </joint>
+        <actuator name="wrist_root4_joint_motor">
+          <hardwareInterface>hardware_interface/EffortJointInterface</hardwareInterface>
+          <mechanicalReduction>1</mechanicalReduction>
+        </actuator>
+    </transmission>
+    <!-- <transmission name="wrist_root4_joint_trans">
+        <plugin>transmission_interface/SimpleTransmission</plugin>
+        <actuator name="wrist_root4_joint_joint" role="actuator1" />
+        <joint name="wrist_root4_joint" role="joint1">
+            <mechanical_reduction>1.0</mechanical_reduction>
+        </joint>
+    </transmission> -->
     <joint name="root4_palm_joint" type="fixed">
         <parent link="root4_link" />

File: src/roboarm_description/urdf/roboarm_ros2_control.xacro (robot description, xacro)
@@ -13,5 +13,4 @@
         <param name="initial_value">0.0</param>
       </state_interface>
-      <state_interface name="velocity" />
     </joint>
     <joint name="body_root1_joint">
@@ -23,5 +22,4 @@
         <param name="initial_value">0.0</param>
       </state_interface>
-      <state_interface name="velocity" />
     </joint>
     <joint name="shoulder_root2_joint">
@@ -33,5 +31,4 @@
         <param name="initial_value">0.0</param>
       </state_interface>
-      <state_interface name="velocity" />
     </joint>
     <joint name="forearm_root3_joint">
@@ -43,5 +40,4 @@
         <param name="initial_value">0.0</param>
       </state_interface>
-      <state_interface name="velocity" />
     </joint>
     <joint name="wrist_root4_joint">
@@ -53,10 +49,8 @@
         <param name="initial_value">0.0</param>
       </state_interface>
-      <state_interface name="velocity" />
     </joint>
     <joint name="palm_left_finger_joint">
       <command_interface name="position" />
       <state_interface name="position" />
-      <state_interface name="velocity" />
     </joint>
     <joint name="palm_right_finger_joint">
@@ -64,5 +58,4 @@
       <param name="multiplier">-1</param>
       <state_interface name="position"/>
-      <state_interface name="velocity" />
     </joint>
   </ros2_control>
