Commit message: fix: add color and joint limits adjustment

File: src/roboarm_description/urdf/roboarm.urdf.xacro (robot description, xacro)
@@ -72,31 +72,4 @@
         </inertial>
     </xacro:macro>
-    <!-- <xacro:macro name="box_inertia" params="m x y z o_xyz o_rpy">
-        <inertial>
-        <mass value="${m}" />
-        <origin xyz="0 0 0" rpy="0 0 0" />
-        <inertia ixx="1.0" ixy="0" ixz="0"
-                 iyy="1.0" iyz="0"
-                 izz="1.0" />
-        </inertial>
-    </xacro:macro>
-    <xacro:macro name="cylinder_inertia" params="m r l o_xyz o_rpy">
-        <inertial>
-            <mass value="${m}" />
-            <origin xyz="0 0 0" rpy="0 0 0" />
-            <inertia ixx="1.0" ixy="0" ixz="0"
-                     iyy="1.0" iyz="0"
-                     izz="1.0" />
-        </inertial>
-    </xacro:macro>
-    <xacro:macro name="sphere_inertia" params="m r o_xyz o_rpy">
-        <inertial>
-            <mass value="${m}" />
-            <origin xyz="${o_xyz}" rpy="${o_rpy}" />
-            <inertia ixx="${(2/5) * m * r * r}" ixy="0" ixz="0"
-                     iyy="${(2/5) * m * r * r}" iyz="0"
-                     izz="${(2/5) * m * r * r}" />
-        </inertial>
-    </xacro:macro> -->
     <!-- Materials -->
     <material name="black">
@@ -153,8 +126,8 @@
         <type>transmission_interface/SimpleTransmission</type>
         <joint name="base_body_joint">
-          <hardwareInterface>hardware_interface/EffortJointInterface</hardwareInterface>
+          <hardwareInterface>hardware_interface/PositionJointInterface</hardwareInterface>
         </joint>
         <actuator name="base_body_joint_motor">
-          <hardwareInterface>hardware_interface/EffortJointInterface</hardwareInterface>
+          <hardwareInterface>hardware_interface/PositionJointInterface</hardwareInterface>
           <mechanicalReduction>1</mechanicalReduction>
         </actuator>
@@ -172,5 +145,5 @@
         <origin xyz="0 ${body_radius} ${body_length - root_radius}" rpy="0 0 0" />
         <axis xyz="0 1 0" />
-        <limit lower="${-pi / 4}" upper="${pi / 4}" velocity="2.0" effort="100"/>
+        <limit lower="${-pi / 2}" upper="${pi / 2}" velocity="2.0" effort="100"/>
         <dynamics damping="${damping}" friction="${friction}"/>
     </joint>
@@ -178,8 +151,8 @@
         <type>transmission_interface/SimpleTransmission</type>
         <joint name="body_root1_joint">
-          <hardwareInterface>hardware_interface/EffortJointInterface</hardwareInterface>
+          <hardwareInterface>hardware_interface/PositionJointInterface</hardwareInterface>
         </joint>
         <actuator name="body_root1_joint_motor">
-          <hardwareInterface>hardware_interface/EffortJointInterface</hardwareInterface>
+          <hardwareInterface>hardware_interface/PositionJointInterface</hardwareInterface>
           <mechanicalReduction>1</mechanicalReduction>
         </actuator>
@@ -202,5 +175,5 @@
         <origin xyz="0 0 ${arm_length - (2 * root_radius)}" rpy="0 0 0" />
         <axis xyz="0 1 0" />
-        <limit lower="${-pi / 4}" upper="${pi / 4}" velocity="2.0" effort="100"/>
+        <limit lower="${-pi / 2}" upper="${pi / 2}" velocity="2.0" effort="100"/>
         <dynamics damping="${damping}" friction="${friction}"/>
     </joint>
@@ -208,8 +181,8 @@
         <type>transmission_interface/SimpleTransmission</type>
         <joint name="shoulder_root2_joint">
-          <hardwareInterface>hardware_interface/EffortJointInterface</hardwareInterface>
+          <hardwareInterface>hardware_interface/PositionJointInterface</hardwareInterface>
         </joint>
         <actuator name="shoulder_root2_joint_motor">
-          <hardwareInterface>hardware_interface/EffortJointInterface</hardwareInterface>
+          <hardwareInterface>hardware_interface/PositionJointInterface</hardwareInterface>
           <mechanicalReduction>1</mechanicalReduction>
         </actuator>
@@ -232,5 +205,5 @@
         <origin xyz="0 0 ${arm_length - (2 * root_radius)}" rpy="0 0 0" />
         <axis xyz="0 1 0" />
-        <limit lower="${-pi / 4}" upper="${pi / 4}" velocity="2.0" effort="100"/>
+        <limit lower="${-pi / 2}" upper="${pi / 2}" velocity="2.0" effort="100"/>
         <dynamics damping="${damping}" friction="${friction}"/>
     </joint>
@@ -238,8 +211,8 @@
         <type>transmission_interface/SimpleTransmission</type>
         <joint name="forearm_root3_joint">
-          <hardwareInterface>hardware_interface/EffortJointInterface</hardwareInterface>
+          <hardwareInterface>hardware_interface/PositionJointInterface</hardwareInterface>
         </joint>
         <actuator name="forearm_root3_joint_motor">
-          <hardwareInterface>hardware_interface/EffortJointInterface</hardwareInterface>
+          <hardwareInterface>hardware_interface/PositionJointInterface</hardwareInterface>
           <mechanicalReduction>1</mechanicalReduction>
         </actuator>
@@ -262,5 +235,5 @@
         <origin xyz="0 ${arm_width / 2} ${(arm_length * 0.5) - root_radius}" rpy="0 0 0" />
         <axis xyz="0 0 1" />
-        <limit lower="${-pi / 2}" upper="${pi / 2}" velocity="2.0" effort="100"/>
+        <limit lower="${-pi}" upper="${pi}" velocity="2.0" effort="100"/>
         <dynamics damping="${damping}" friction="${friction}"/>
     </joint>
@@ -268,8 +241,8 @@
         <type>transmission_interface/SimpleTransmission</type>
         <joint name="wrist_root4_joint">
-          <hardwareInterface>hardware_interface/EffortJointInterface</hardwareInterface>
+          <hardwareInterface>hardware_interface/PositionJointInterface</hardwareInterface>
         </joint>
         <actuator name="wrist_root4_joint_motor">
-          <hardwareInterface>hardware_interface/EffortJointInterface</hardwareInterface>
+          <hardwareInterface>hardware_interface/PositionJointInterface</hardwareInterface>
           <mechanicalReduction>1</mechanicalReduction>
         </actuator>
@@ -294,4 +267,14 @@
         <limit lower="0" upper="${(arm_width * 3 / 2) - (arm_width * 0.5)}" velocity="2.0" effort="100"/>
     </joint>
+    <transmission name="palm_left_finger_joint_trans">
+        <type>transmission_interface/SimpleTransmission</type>
+        <joint name="palm_left_finger_joint">
+          <hardwareInterface>hardware_interface/PositionJointInterface</hardwareInterface>
+        </joint>
+        <actuator name="palm_left_finger_joint_motor">
+          <hardwareInterface>hardware_interface/PositionJointInterface</hardwareInterface>
+          <mechanicalReduction>1</mechanicalReduction>
+        </actuator>
+    </transmission>
     <joint name="palm_right_finger_joint" type="prismatic">
         <parent link="palm_link" />

File: src/roboarm_description/urdf/roboarm_gazebo.xacro (robot description, xacro)
@@ -2,9 +2,46 @@
 <robot xmlns:xacro="http://www.ros.org/wiki/xacro" name="roboarm">
     <gazebo>
-    <plugin filename="libgazebo_ros2_control.so" name="gazebo_ros2_control">
-        <robot_param>robot_description</robot_param>
-        <robot_param_node>robot_state_publisher</robot_param_node>
-        <parameters>$(find roboarm_controller)/config/roboarm_controller.yaml</parameters>
-    </plugin>
+        <plugin filename="libgazebo_ros2_control.so" name="gazebo_ros2_control">
+            <robot_param>robot_description</robot_param>
+            <robot_param_node>robot_state_publisher</robot_param_node>
+            <parameters>$(find roboarm_controller)/config/roboarm_controller.yaml</parameters>
+        </plugin>
+    </gazebo>
+    <!-- Adding colors to robot part as in gazebo classic tag material doesnt work -->
+    <gazebo reference="base_link">
+        <material>Gazebo/Black</material>
+    </gazebo>
+    <gazebo reference="body_link">
+        <material>Gazebo/Orange</material>
+    </gazebo>
+    <gazebo reference="shoulder_link">
+        <material>Gazebo/Orange</material>
+    </gazebo>
+    <gazebo reference="forearm_link">
+        <material>Gazebo/Orange</material>
+    </gazebo>
+    <gazebo reference="wrist_link">
+        <material>Gazebo/Orange</material>
+    </gazebo>
+    <gazebo reference="palm_link">
+        <material>Gazebo/Yellow</material>
+    </gazebo>
+    <gazebo reference="left_finger_link">
+        <material>Gazebo/Yellow</material>
+    </gazebo>
+    <gazebo reference="right_finger_link">
+        <material>Gazebo/Yellow</material>
+    </gazebo>
+    <gazebo reference="root1_link">
+        <material>Gazebo/DarkGrey</material>
+    </gazebo>
+    <gazebo reference="root2_link">
+        <material>Gazebo/DarkGrey</material>
+    </gazebo>
+    <gazebo reference="root3_link">
+        <material>Gazebo/DarkGrey</material>
+    </gazebo>
+    <gazebo reference="root4_link">
+        <material>Gazebo/DarkGrey</material>
     </gazebo>
 </robot>

File: src/roboarm_description/urdf/roboarm_ros2_control.xacro (robot description, xacro)
@@ -10,7 +10,9 @@
         <param name="max">${pi / 2}</param>
       </command_interface>
+      <!-- <command_interface name="velocity" /> -->
       <state_interface name="position">
         <param name="initial_value">0.0</param>
       </state_interface>
+      <!-- <state_interface name="velocity" /> -->
     </joint>
     <joint name="body_root1_joint">
@@ -19,7 +21,9 @@
         <param name="max">${pi / 2}</param>
       </command_interface>
+      <!-- <command_interface name="velocity" /> -->
       <state_interface name="position">
         <param name="initial_value">0.0</param>
       </state_interface>
+      <!-- <state_interface name="velocity" /> -->
     </joint>
     <joint name="shoulder_root2_joint">
@@ -28,7 +32,9 @@
         <param name="max">${pi / 2}</param>
       </command_interface>
+      <!-- <command_interface name="velocity" /> -->
       <state_interface name="position">
         <param name="initial_value">0.0</param>
       </state_interface>
+      <!-- <state_interface name="velocity" /> -->
     </joint>
     <joint name="forearm_root3_joint">
@@ -37,7 +43,9 @@
         <param name="max">${pi / 2}</param>
       </command_interface>
+      <!-- <command_interface name="velocity" /> -->
       <state_interface name="position">
         <param name="initial_value">0.0</param>
       </state_interface>
+      <!-- <state_interface name="velocity" /> -->
     </joint>
     <joint name="wrist_root4_joint">
@@ -46,7 +54,9 @@
         <param name="max">${pi / 2}</param>
       </command_interface>
+      <!-- <command_interface name="velocity" /> -->
       <state_interface name="position">
         <param name="initial_value">0.0</param>
       </state_interface>
+      <!-- <state_interface name="velocity" /> -->
     </joint>
     <joint name="palm_left_finger_joint">

Commit message: fix: add slider control feature

File: src/roboarm_description/urdf/roboarm.urdf.xacro (robot description, xacro)
@@ -121,5 +121,5 @@
         <axis xyz="0 0 1" />
         <dynamics damping="${damping}" friction="${friction}"/>
-        <limit lower="${-pi / 2}" upper="${pi / 2}" velocity="2.0" effort="100"/>
+        <limit lower="${-pi}" upper="${pi}" velocity="2.0" effort="100"/>
     </joint>
     <transmission name="base_body_joint_trans">
@@ -235,5 +235,5 @@
         <origin xyz="0 ${arm_width / 2} ${(arm_length * 0.5) - root_radius}" rpy="0 0 0" />
         <axis xyz="0 0 1" />
-        <limit lower="${-pi}" upper="${pi}" velocity="2.0" effort="100"/>
+        <limit lower="${-pi / 2}" upper="${pi / 2}" velocity="2.0" effort="100"/>
         <dynamics damping="${damping}" friction="${friction}"/>
     </joint>

Commit message: fix: before switching to gripper effort

File: src/roboarm_description/urdf/roboarm.urdf.xacro (robot description, xacro)
@@ -52,4 +52,31 @@
                     <box size="${x} ${y} ${z}" />
                 </geometry>
+                <origin xyz="${ox} ${oy} ${oz}" rpy="0 0 0" />
+            </collision>
+        </link>
+    </xacro:macro>
+    <xacro:macro name="finger_link" params="name x y z ox oy oz mass material">
+        <link name="${name}_link">
+            <visual>
+                <geometry>
+                    <box size="${x} ${y} ${z}" />
+                </geometry>
+                <origin xyz="${ox} ${oy} ${oz}" rpy="0 0 0" />
+                <material name="${material}" />
+            </visual>
+            <xacro:box_inertia m="10.0" x="${x}" y="${y}" z="${z}" o_xyz="${ox} ${oy} ${oz}" o_rpy="0 0 0" />
+            <collision>
+                <geometry>
+                    <box size="${x} ${y} ${z}" />
+                </geometry>
+                <surface>
+                    <friction>
+                        <ode>
+                        <!-- Основные коэффициенты трения -->
+                        <mu>1.2</mu>    <!-- Статическое трение (увеличьте для лучшего захвата) -->
+                        <mu2>1.0</mu2>  <!-- Динамическое трение -->
+                        </ode>
+                    </friction>
+                </surface>
                 <origin xyz="${ox} ${oy} ${oz}" rpy="0 0 0" />
             </collision>
@@ -108,7 +135,7 @@
     <xacro:box_link name="palm" x="${arm_width * 3}" y="${arm_width}" z="${arm_width}" ox="0" oy="0" oz="${arm_width / 2}" mass="${arm_mass}" material="orange" />
     <!-- Making left_finger_link -->
-    <xacro:box_link name="left_finger" x="${arm_width * 0.5}" y="${arm_width * 0.5}" z="${arm_width * 4}" ox="0" oy="0" oz="${arm_width * 4 / 2}" mass="0.001" material="orange" />
+    <xacro:finger_link name="left_finger" x="${arm_width * 0.5}" y="${arm_width * 0.5}" z="${arm_width * 4}" ox="0" oy="0" oz="${arm_width * 4 / 2}" mass="0.001" material="orange" />
     <!-- Making right_finger_link -->
-    <xacro:box_link name="right_finger" x="${arm_width * 0.5}" y="${arm_width * 0.5}" z="${arm_width * 4}" ox="0" oy="0" oz="${arm_width * 4 / 2}" mass="0.001" material="orange" />
+    <xacro:finger_link name="right_finger" x="${arm_width * 0.5}" y="${arm_width * 0.5}" z="${arm_width * 4}" ox="0" oy="0" oz="${arm_width * 4 / 2}" mass="0.001" material="orange" />
     <!-- Joints -->
     <joint name="world_base_joint" type="fixed">
@@ -284,5 +311,5 @@
         <origin xyz="${(arm_width * 3 / 2) - (arm_width * 0.5 / 2)} 0 ${arm_width}" rpy="0 0 0" />
         <axis xyz="1 0 0" />
-        <limit lower="${-(arm_width * 3 / 2) + (arm_width * 0.5)}" upper="0" velocity="2.0" effort="100"/>
+        <limit lower="${-(arm_width * 3 / 2) + (arm_width * 0.5)}" upper="0" velocity="2.0" effort="20"/>
         <mimic joint="palm_left_finger_joint" multiplier="-1" />
     </joint>
