Commit message: fix: correctly bridge gz camera to ros

File: src/roboarm_description/urdf/camera.xacro (robot description, xacro)
@@ -19,11 +19,11 @@
         <origin xyz="0 0 0" rpy="${-pi/2} 0 ${-pi/2}"/>
     </joint>
-    <link name="camera_link_optical"></link>
+    <link name="camera_link_optical"/>
     <gazebo reference="camera_link">
         <material>Gazebo/Red</material>
         <sensor name="camera" type="camera">
-            <pose> 0 0 0 0 0 0 </pose>
+            <pose>0 0 0 0 0 0</pose>
             <visualize>true</visualize>
-            <update_rate>10</update_rate>
+            <update_rate>30</update_rate>
             <camera>
                 <horizontal_fov>1.089</horizontal_fov>
@@ -38,6 +38,13 @@
                 </clip>
             </camera>
+            <!-- libgazebo_ros_camera_system.so dont create ros topics -->
             <plugin name="camera_controller" filename="libgazebo_ros_camera.so">
+                <ros>
+                    <namespace>/roboeye</namespace>
+                </ros>
                 <frame_name>camera_link_optical</frame_name>
+                <camera_name>camera</camera_name>
+                <image_topic_name>image_raw</image_topic_name>
+                <camera_info_topic_name>camera_info</camera_info_topic_name>
             </plugin>
         </sensor>

Commit message: feat: reacher train ddpg

File: src/roboarm_description/urdf/camera.xacro (robot description, xacro)
@@ -2,7 +2,7 @@
 <robot xmlns:xacro="http://www.ros.org/wiki/xacro" name="roboarm">
     <joint name="camera_joint" type="fixed">
-        <parent link="palm_link"/>
+        <parent link="wrist_link"/>
         <child link="camera_link"/>
-        <origin xyz="0 0.2 0" rpy="0 ${-pi/2} 0"/>
+        <origin xyz="-0.2 0.025 0.225" rpy="0 ${-pi/2} 0"/>
     </joint>
     <link name="camera_link">

File: src/roboarm_description/urdf/roboarm.urdf.xacro (robot description, xacro)
@@ -13,5 +13,5 @@
     <xacro:property name="base_height" value="0.1" />
     <xacro:property name="body_radius" value="0.1" />
-    <xacro:property name="body_length" value="0.4" />
+    <xacro:property name="body_length" value="0.6" />
     <xacro:property name="root_radius" value="0.05" />
     <xacro:property name="root_length" value="0.05" />

Commit message: feat: docstrings

File: src/roboarm_description/urdf/camera.xacro (robot description, xacro)
@@ -2,7 +2,9 @@
 <robot xmlns:xacro="http://www.ros.org/wiki/xacro" name="roboarm">
     <joint name="camera_joint" type="fixed">
-        <parent link="wrist_link"/>
+        <parent link="base_link"/>
         <child link="camera_link"/>
-        <origin xyz="-0.2 0.025 0.225" rpy="0 ${-pi/2} 0"/>
+        <origin xyz="1.0 -1.0 3.0" rpy="0 ${pi/2} 0"/>
+        <!-- <origin xyz="0 0 1.0" rpy="0 0.523599 0"/> -->
+        <!-- <origin xyz="-0.2 0.025 0.225" rpy="0 ${-pi/2} 0"/> -->
     </joint>
     <link name="camera_link">
@@ -28,8 +30,12 @@
             <camera>
                 <horizontal_fov>1.089</horizontal_fov>
+                <!-- 1.089 - default -->
+                <!-- 1.047 - 60 -->
+                <!-- 1.571 - 90 -->
+                <!-- 2.094 - 120 -->
                 <image>
                     <format>R8G8B8</format>
                     <width>640</width>
-                    <height>480</height>
+                    <height>640</height>
                 </image>
                 <clip>
